File: universal pcb/universal pcb.kicad_pcb (KiCad board)
At the start: 2 copper layers, 30 x 22.5 mm, 6 parts

Commit message: create front panel for prototype, save kicad
Parts:
- REF** (x2): footprint Connector_PinHeader_2.54mm:PinHeader_1x08_P2.54mm_Vertical -> Eurorack:PinHeader_1x08_P2.54mm_Vertical
